File: ECAD/PCBs/Specialty/UFC3/UFC_3.0.sch (KiCad schematic (older format))
At the start: 426 parts, among them J1 PWR IN, J2 OLED DISP, J3 PANEL SW, J7 HUD BIT, J8 AP BTNS, J9 HUD PANL, P1 CONN_01X01, P10 PWM, P11 Analog, P12 Communication, P13 Digital, P2 CONN_01X01, P3 CONN_01X01, P4 CONN_01X01, P5 CONN_01X01, P6 CONN_01X01, P7 PWM, P8 Power, P9 Analog, SW1 1, SW10 8, SW11 9, SW12 OPT4, SW13 CLR, SW14 ~0, SW15 ENT, SW16 OPT5, SW17 OPT1, SW18 I/P, SW19 EMCON, SW2 2, SW3 3, SW4 OPT2, SW5 4, SW6 5, SW7 6, SW8 OPT3, SW9 7, U1 MAX6955AAX+, U2 TXS0102DCT, U3 MAX6955AAX+, U4 MAX6955AAX+

Commit message: temporary commit, this commit contains a partial version of the routing for UFC v3. along this commit I have added a python script to place the components based on the location listed on a csv file
Parts:
- removed MK1, MK2, MK3, MK4: Mounting_Hole, Mounting_Holes:MountingHole_4.3mm_M4, symbol Mechanical:MountingHole
- removed P1, P2, P3, P4, P5, P6: CONN_01X01, Socket_Arduino_Mega:Arduino_1pin, symbol Connector_Generic:Conn_01x01
- added M5, M6, M7, M8: mounting hole, MountingHole:MountingHole_2.7mm_M2.5, symbol Mechanical:MountingHole
- added R9: 56k, Resistor_SMD:R_0402_1005Metric, symbol Device:R
- P10, P11, P12, P8, P9: footprint Socket_Arduino_Mega:Socket_Strip_Arduino_1x08 -> Connector_PinHeader_2.54mm:PinHeader_1x08_P2.54mm_Vertical_SMD_Pin1Left
- P13: footprint Socket_Arduino_Mega:Socket_Strip_Arduino_2x18 -> Connector_PinHeader_2.54mm:PinHeader_2x18_P2.54mm_Vertical_SMD
- P7: footprint Socket_Arduino_Mega:Socket_Strip_Arduino_1x10 -> Connector_PinHeader_2.54mm:PinHeader_1x10_P2.54mm_Vertical_SMD_Pin1Left
- SW1, SW10, SW11, SW13, SW14, SW15, SW18, SW19, SW2, SW3, SW5, SW6, SW7, SW9: footprint KiCAD Libraries:SWITCH_SNAP_DOME_6.3mm_DIA_SINGLE_SIDE_PCB -> KiCAD Libraries:SWITCH_SNAP_DOME
- SW12: value OPT4 -> OPT3; footprint KiCAD Libraries:SWITCH_SNAP_DOME_6.3mm_DIA_SINGLE_SIDE_PCB -> KiCAD Libraries:SWITCH_SNAP_DOME
- SW16: value OPT5 -> OPT4; footprint KiCAD Libraries:SWITCH_SNAP_DOME_6.3mm_DIA_SINGLE_SIDE_PCB -> KiCAD Libraries:SWITCH_SNAP_DOME
- SW17: value OPT1 -> OPT5; footprint KiCAD Libraries:SWITCH_SNAP_DOME_6.3mm_DIA_SINGLE_SIDE_PCB -> KiCAD Libraries:SWITCH_SNAP_DOME
- SW4: value OPT2 -> OPT1; footprint KiCAD Libraries:SWITCH_SNAP_DOME_6.3mm_DIA_SINGLE_SIDE_PCB -> KiCAD Libraries:SWITCH_SNAP_DOME
- SW8: value OPT3 -> OPT2; footprint KiCAD Libraries:SWITCH_SNAP_DOME_6.3mm_DIA_SINGLE_SIDE_PCB -> KiCAD Libraries:SWITCH_SNAP_DOME
- renumbered C9 to C10, C7 to C4, C10 to C5, C4 to C6, C5 to C7, C6 to C8, C8 to C9, D137 to D129, D138 to D130, D139 to D131, D140 to D132, D141 to D133, D142 to D134, D143 to D135, D144 to D136, D145 to D137, D146 to D138, D147 to D139, D148 to D140, D149 to D141, D150 to D142, D151 to D143, D152 to D144, D153 to D145, D154 to D146, D155 to D147, D156 to D148, D157 to D149, D158 to D150, D159 to D151, D160 to D152, D161 to D153, D162 to D154, D163 to D155, D164 to D156, D165 to D157, D166 to D158, D167 to D159, D168 to D160, D171 to D161, D172 to D162, D173 to D163, D174 to D164, D175 to D165, D176 to D166, D177 to D167, D178 to D168, D179 to D169, D180 to D170, D181 to D171, D182 to D172, D183 to D173, D184 to D174, D185 to D175, D186 to D176, D187 to D177, D188 to D178, D189 to D179, D190 to D180, D191 to D181, D192 to D182, D193 to D183, D194 to D184, D195 to D185, D196 to D186, D197 to D187, D198 to D188, D199 to D189, D200 to D190, D201 to D191, D202 to D192, D203 to D193, D204 to D194, D205 to D195, D206 to D196, D207 to D197, D208 to D198, D209 to D199, D210 to D200, D211 to D201, D212 to D202, D213 to D203, D214 to D204, D215 to D205, D216 to D206, D217 to D207, D218 to D208, D219 to D209, D220 to D210, D221 to D211, D222 to D212, D223 to D213, D224 to D214, D225 to D215, D226 to D216, D227 to D217, D228 to D218, D229 to D219, D230 to D220, D231 to D221, D232 to D222, D233 to D223, D234 to D224, D235 to D225, D236 to D226, D237 to D227, D238 to D228, D239 to D229, D240 to D230, D241 to D231, D242 to D232, D243 to D233, D244 to D234, D245 to D235, D246 to D236, D247 to D237, D248 to D238, D249 to D239, D250 to D240, D251 to D241, D252 to D242, D253 to D243, D254 to D244, D255 to D245, D256 to D246, D257 to D247, D258 to D248, D259 to D249, D260 to D250, D261 to D251, D262 to D252, D263 to D253, D264 to D254, D265 to D255, D266 to D256, D267 to D257, D268 to D258, D269 to D259, D270 to D260, D271 to D261, D272 to D262, D273 to D263, D274 to D264, D275 to D265, D276 to D266, D277 to D267, D278 to D268, D279 to D269, D280 to D270, D281 to D271, D282 to D272, D283 to D273, D284 to D274, D285 to D275, D286 to D276, D287 to D277, D288 to D278, D289 to D279, D290 to D280, D291 to D281, D292 to D282, D293 to D283, D294 to D284, D295 to D285, D296 to D286, D297 to D287, D298 to D288, D299 to D289, D300 to D290, D301 to D291, D302 to D292, D303 to D293, D304 to D294, D305 to D295, D306 to D296, D307 to D297, D308 to D298, D309 to D299, D310 to D300, D311 to D301, D312 to D302, D313 to D303, D314 to D304, D315 to D305, D316 to D306, D317 to D307, D318 to D308, D319 to D309, D320 to D310, D321 to D311, D322 to D312, D323 to D313, D324 to D314, D325 to D315, D326 to D316, D327 to D317, D328 to D318, D329 to D319, D330 to D320, D331 to D321, D332 to D322, D333 to D323, D334 to D324, D335 to D325, D336 to D326, D337 to D327, D338 to D328, D339 to D329, D340 to D330, D341 to D331, D342 to D332, D343 to D333, D344 to D334, D345 to D335, D346 to D336, D347 to D337, D348 to D338, D349 to D339, D350 to D340, D351 to D341, D352 to D342, D353 to D343, D354 to D344, D355 to D345, D356 to D346, D357 to D347, D358 to D348, D359 to D349, D360 to D350, D361 to D351, D362 to D352, J7 to J4, J8 to J5, J9 to J6, D129 to opt0-1, D130 to opt0-2, D131 to opt1-1, D132 to opt1-2, D133 to opt2-1, D134 to opt2-2, D135 to opt3-1, D136 to opt3-2, D169 to opt4-1, D170 to opt4-2
Connections:
- wire segments 1026 -> 1025
- no-connect marks 69 -> 62
Other:
- note added: "IMPORTANT NOTE:\nThe arduino connector is designed for Arduino Mega to be connected on the Front of the arduino...\nThis board assumes the connector is on the back. this requires the existing Arduino connectors to be removed and soldered on the other side of the arduino board"
- note added: "OE is controlled via A10"
- note removed: "MOUNTING HOLES"
- moved on the sheet: SW1, SW10, SW11, SW12, SW13, SW14, SW15, SW16, SW17, SW2, SW3, SW4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
